File: LPF.kicad_sch (KiCad schematic)
At the start: 31 parts, among them U4 OPA1679

Commit message: First order
Parts:
- U4: LCSC C1849432 -> C1849432
Changed lines of the file:
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@@
 			)
 		)
-		(property "LCSC" "C1849432 "
+		(property "LCSC" "C1849432"
 			(at 128.27 166.37 0)
 			(effects
@@
 			)
 		)
-		(property "LCSC" "C1849432 "
+		(property "LCSC" "C1849432"
 			(at 128.27 90.17 0)
 			(effects
@@
 			)
 		)
-		(property "LCSC" "C1849432 "
+		(property "LCSC" "C1849432"
 			(at 128.27 52.07 0)
 			(effects
@@
 			)
 		)
-		(property "LCSC" "C1849432 "
+		(property "LCSC" "C1849432"
 			(at 128.27 52.07 0)
 			(effects
@@
 			)
 		)
-		(property "LCSC" "C1849432 "
+		(property "LCSC" "C1849432"
 			(at 128.27 129.54 0)
 			(effects

Commit message: Updated LCSC parts number for unmatched footprint
Parts:
- U4: footprint Package_DFN_QFN:WQFN-16-1EP_4x4mm_P0.5mm_EP2.6x2.6mm -> Package_DFN_QFN:QFN-16-1EP_4x4mm_P0.65mm_EP2.1x2.1mm
Changed lines of the file:
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@@
 			)
 		)
-		(property "Footprint" "Package_DFN_QFN:WQFN-16-1EP_4x4mm_P0.5mm_EP2.6x2.6mm"
+		(property "Footprint" "Package_DFN_QFN:QFN-16-1EP_4x4mm_P0.65mm_EP2.1x2.1mm"
 			(at 127 168.91 0)
 			(effects
@@
 			)
 		)
-		(property "Footprint" "Package_DFN_QFN:WQFN-16-1EP_4x4mm_P0.5mm_EP2.6x2.6mm"
+		(property "Footprint" "Package_DFN_QFN:QFN-16-1EP_4x4mm_P0.65mm_EP2.1x2.1mm"
 			(at 127 92.71 0)
 			(effects
@@
 			)
 		)
-		(property "Footprint" "Package_DFN_QFN:WQFN-16-1EP_4x4mm_P0.5mm_EP2.6x2.6mm"
+		(property "Footprint" "Package_DFN_QFN:QFN-16-1EP_4x4mm_P0.65mm_EP2.1x2.1mm"
 			(at 127 54.61 0)
 			(effects
@@
 			)
 		)
-		(property "Footprint" "Package_DFN_QFN:WQFN-16-1EP_4x4mm_P0.5mm_EP2.6x2.6mm"
+		(property "Footprint" "Package_DFN_QFN:QFN-16-1EP_4x4mm_P0.65mm_EP2.1x2.1mm"
 			(at 127 49.53 0)
 			(effects
@@
 			)
 		)
-		(property "Footprint" "Package_DFN_QFN:WQFN-16-1EP_4x4mm_P0.5mm_EP2.6x2.6mm"
+		(property "Footprint" "Package_DFN_QFN:QFN-16-1EP_4x4mm_P0.65mm_EP2.1x2.1mm"
 			(at 127 132.08 0)
 			(effects
